File: uHoubolt_PCB_GNSS.kicad_pcb (KiCad board)
At the start: 2 copper layers, 90 x 90 mm, 5 parts, among them J1 UART, U1 SAM-M8Q

Commit message: first revision done
Parts:
- added C4: 470m, Capacitor_SMD:CP_Elec_10x10.5, B.Cu at (150.0, 110.8)
- added D1: Schottky, Diode_SMD:D_SOD-123F, B.Cu at (143.4, 103.9)
- added H1: M3, MountingHole:MountingHole_3.2mm_M3_Pad_Via, F.Cu at (176.9, 73.1)
- added H2: M3, MountingHole:MountingHole_3.2mm_M3_Pad_Via, F.Cu at (123.1, 73.1)
- added H3: M3, MountingHole:MountingHole_3.2mm_M3_Pad_Via, F.Cu at (123.1, 126.9)
- added H4: M3, MountingHole:MountingHole_3.2mm_M3_Pad_Via, F.Cu at (176.9, 126.9)
- added J2: GND, TestPoint:TestPoint_Pad_4.0x4.0mm, B.Cu at (185.9, 100.0)
- added J3: ANT, TestPoint:TestPoint_THTPad_D1.5mm_Drill0.7mm, B.Cu at (191.1, 100.0)
- added R1: 330, Resistor_SMD:R_0603_1608Metric, B.Cu at (143.4, 107.7)
Connections:
- C3 pad 1: +3V3 -> Net-(C3-Pad1)
- U1 pad 3: +3V3 -> Net-(C3-Pad1)
Routing:
- net Net-(C3-Pad1): track 0.00 -> 12.3 mm, vias 0 -> 1
- net Net-(D1-Pad1): track 0.00 -> 1.58 mm
- net +3V3: track 32.9 -> 31.7 mm
- net GND: vias 0 -> 54
Other:
- board size 90 x 90 mm -> 85 x 85 mm
- board text added: "GND RxD TxD 3V3"

Commit message: Update footprints and fixed minor naming fails.
Parts:
- added C10: 100n, Capacitor_SMD:C_0603_1608Metric, B.Cu at (223.1, 41.7)
- added C11: 100n, Capacitor_SMD:C_0603_1608Metric, B.Cu at (242.1, 67.4)
- added C12: 2u2, Capacitor_SMD:C_0603_1608Metric, B.Cu at (200.6, 31.9)
- added C13: 100n, Capacitor_SMD:C_0603_1608Metric, B.Cu at (70.5, 188.6)
- added C14: 100n, Capacitor_SMD:C_0603_1608Metric, B.Cu at (39.5, 189.9)
- added C15: 2u2, Capacitor_SMD:C_0603_1608Metric, B.Cu at (99.2, 34.2)
- added C16: 100n, Capacitor_SMD:C_0603_1608Metric, B.Cu at (74.8, 188.6)
- added C17: 100n, Capacitor_SMD:C_0603_1608Metric, B.Cu at (43.1, 189.9)
- added C18: 10u, Capacitor_SMD:C_0603_1608Metric, B.Cu at (143.5, 71.3)
- added C19: 100n, Capacitor_SMD:C_0603_1608Metric, B.Cu at (143.5, 73.1)
- added C20: 100n, Capacitor_SMD:C_0603_1608Metric, B.Cu at (227.7, 57.7)
- added C21: 100n, Capacitor_SMD:C_0603_1608Metric, B.Cu at (205.4, 37.0)
- added C22: 100n, Capacitor_SMD:C_0603_1608Metric, B.Cu at (142.4, 79.7)
- added C23: 22u, Capacitor_SMD:C_0603_1608Metric, B.Cu at (151.0, 73.8)
- added C24: 22u, Capacitor_SMD:C_0603_1608Metric, B.Cu at (152.8, 73.8)
- added C25: 2u2, Capacitor_SMD:C_0603_1608Metric, B.Cu at (225.2, 47.7)
- added C26: 2u2, Capacitor_SMD:C_0603_1608Metric, B.Cu at (231.7, 57.7)
- added C27: 2u2, Capacitor_SMD:C_0603_1608Metric, B.Cu at (246.1, 67.4)
- added C28: 100n, Capacitor_SMD:C_0603_1608Metric, B.Cu at (201.9, 29.4)
- added C29: 22u, Capacitor_SMD:C_0603_1608Metric, B.Cu at (223.2, 50.2)
- added C30: 100n, Capacitor_SMD:C_0603_1608Metric, B.Cu at (209.4, 37.0)
- added C31: 100n, Capacitor_SMD:C_0603_1608Metric, B.Cu at (227.2, 52.7)
- added C32: 100n, Capacitor_SMD:C_0603_1608Metric, B.Cu at (215.7, 44.2)
- added C33: 100n, Capacitor_SMD:C_0603_1608Metric, B.Cu at (213.4, 37.0)
- added C34: 100n, Capacitor_SMD:C_0603_1608Metric, B.Cu at (223.7, 44.2)
- added C5: 2u2, Capacitor_SMD:C_0603_1608Metric, B.Cu at (208.6, 32.0)
- added C6: 100n, Capacitor_SMD:C_0603_1608Metric, B.Cu at (205.9, 29.4)
- added C7: 100n, Capacitor_SMD:C_0603_1608Metric, B.Cu at (246.1, 64.9)
- added C8: 100n, Capacitor_SMD:C_0603_1608Metric, B.Cu at (26.8, 18.2)
- added C9: 100n, Capacitor_SMD:C_0603_1608Metric, B.Cu at (201.9, 26.9)
- added D2: CDBU0240-HF, Diode_SMD:D_SOD-323F, B.Cu at (250.1, 39.1)
- added D3: 5V, LED_SMD:LED_0201_0603Metric, B.Cu at (197.1, 31.5)
- added D4: TVS 3V3, TXV_Library_Footprints:SOD882D, B.Cu at (202.2, 37.2)
- added D5: 3V3, LED_SMD:LED_0201_0603Metric, B.Cu at (204.5, 39.1)
- added F1: 500mA, Fuse:Fuse_0603_1608Metric, B.Cu at (154.6, 73.8)
- added J10: CAN1, Connector_JST:JST_GH_BM04B-GHS-TBT_1x04-1MP_P1.25mm_Vertical, B.Cu at (166.3, 124.6)
- added J11: CAN1, Connector_JST:JST_GH_BM04B-GHS-TBT_1x04-1MP_P1.25mm_Vertical, B.Cu at (133.6, 131.8)
- added J12: MMCX-J-P-H-ST-SM1, TXV_Library_Footprints:SAMTEC_MMCX-J-P-H-ST-SM1, B.Cu at (239.7, 15.9)
- added J4: CAN1, Connector_JST:JST_GH_BM04B-GHS-TBT_1x04-1MP_P1.25mm_Vertical, B.Cu at (156.1, 124.6)
- added J5: CAN1, Connector_JST:JST_GH_BM04B-GHS-TBT_1x04-1MP_P1.25mm_Vertical, B.Cu at (143.8, 124.4)
- added J6: CAN1, Connector_JST:JST_GH_BM04B-GHS-TBT_1x04-1MP_P1.25mm_Vertical, B.Cu at (166.3, 132.0)
- added J7: CAN1, Connector_JST:JST_GH_BM04B-GHS-TBT_1x04-1MP_P1.25mm_Vertical, B.Cu at (133.6, 124.4)
- added J8: CAN1, Connector_JST:JST_GH_BM04B-GHS-TBT_1x04-1MP_P1.25mm_Vertical, B.Cu at (156.1, 132.0)
- added J9: CAN1, Connector_JST:JST_GH_BM04B-GHS-TBT_1x04-1MP_P1.25mm_Vertical, B.Cu at (143.8, 131.8)
- added JP1: SolderJumper_, Jumper:SolderJumper-2_P1.3mm_Open_Pad1.0x1.5mm, B.Cu at (176.4, 20.8)
- added L1: 4u7, TXV_Library_Footprints:SRN4018TA-4R7M, B.Cu at (147.7, 76.4)
- added LED1: LED_Small_Filled, LED_SMD:LED_0603_1608Metric, B.Cu at (254.5, 45.4)
- added LED2: LED_Small_Filled, LED_SMD:LED_0603_1608Metric, B.Cu at (258.6, 45.4)
- added LS1: Speaker, TXV_Library_Footprints:Piezo_Buzzer, B.Cu at (166.0, 74.6)
- added Q1: SISA88DN or similar, TXV_Library_Footprints:PowerPAK_1212-8, B.Cu at (226.2, 31.4)
- added R10: 120, Resistor_SMD:R_0603_1608Metric, B.Cu at (67.7, 192.5)
- added R11: 120, Resistor_SMD:R_0603_1608Metric, B.Cu at (36.7, 194.0)
- added R12: R_x, Resistor_SMD:R_0603_1608Metric, B.Cu at (151.0, 77.1)
- added R13: R_y, Resistor_SMD:R_0603_1608Metric, B.Cu at (152.8, 77.1)
- added R14: 1k, Resistor_SMD:R_0603_1608Metric, B.Cu at (235.7, 61.3)
- added R15: 10k, Resistor_SMD:R_0603_1608Metric, B.Cu at (227.2, 50.2)
- added R16: 10k, Resistor_SMD:R_0603_1608Metric, B.Cu at (234.1, 63.8)
- added R17: 120, Resistor_SMD:R_0603_1608Metric, B.Cu at (204.6, 31.9)
- added R2: 120, Resistor_SMD:R_0603_1608Metric, B.Cu at (231.2, 50.2)
- added R3: 120, Resistor_SMD:R_0603_1608Metric, B.Cu at (239.7, 57.5)
- added R4: 120, Resistor_SMD:R_0603_1608Metric, B.Cu at (217.2, 46.7)
- added R5: 1k, Resistor_SMD:R_0603_1608Metric, B.Cu at (235.7, 58.8)
- added R6: 1k, Resistor_SMD:R_0603_1608Metric, B.Cu at (235.7, 56.3)
- added R7: 56k, Resistor_SMD:R_0603_1608Metric, B.Cu at (229.2, 47.7)
- added R8: 10k, Resistor_SMD:R_0603_1608Metric, B.Cu at (197.9, 29.4)
- added R9: 100, Resistor_SMD:R_0603_1608Metric, B.Cu at (212.6, 32.0)
- added SuperCap1: 1F, Capacitor_SMD:CP_Elec_10x10.5, B.Cu at (150.0, 100.0)
- added TP1: TestPoint_Probe, TestPoint:TestPoint_Pad_D1.0mm, B.Cu at (194.4, 27.1)
- added TP10: TestPoint_Probe, TestPoint:TestPoint_Pad_D1.0mm, B.Cu at (223.7, 55.5)
- added TP11: TestPoint_Probe, TestPoint:TestPoint_Pad_D1.0mm, B.Cu at (212.1, 44.8)
- added TP12: TestPoint_Probe, TestPoint:TestPoint_Pad_D1.0mm, B.Cu at (230.6, 63.5)
- added TP2: TestPoint_Probe, TestPoint:TestPoint_Pad_D1.0mm, B.Cu at (215.7, 49.5)
- added TP3: TestPoint_Probe, TestPoint:TestPoint_Pad_D1.0mm, B.Cu at (219.7, 52.0)
- added TP4: TestPoint_Probe, TestPoint:TestPoint_Pad_D1.0mm, B.Cu at (220.6, 55.5)
- added TP5: TestPoint_Probe, TestPoint:TestPoint_Pad_D1.0mm, B.Cu at (201.9, 34.7)
- added TP6: TestPoint_Probe, TestPoint:TestPoint_Pad_D1.0mm, B.Cu at (228.2, 60.5)
- added TP7: TestPoint_Probe, TestPoint:TestPoint_Pad_D1.0mm, B.Cu at (224.2, 58.5)
- added TP8: TestPoint_Probe, TestPoint:TestPoint_Pad_D1.0mm, B.Cu at (234.6, 66.6)
- added TP9: TestPoint_Probe, TestPoint:TestPoint_Pad_D1.0mm, B.Cu at (207.5, 39.8)
- added U11: LPS25HB, Package_LGA:ST_HLGA-10_2.5x2.5mm_P0.6mm_LayoutBorder3x2y, B.Cu at (250.2, 65.7)
- added U2: STM32G491MET6-LQFP80, Package_QFP:LQFP-80_12x12mm_P0.5mm, B.Cu at (170.3, 92.1)
- added U3: W25Q256JV, TXV_Library_Footprints:WSON-8-8x6mm, B.Cu at (171.6, 108.4)
- added U4: MCP1700-3302E, Package_TO_SOT_SMD:SOT-23, B.Cu at (96.2, 34.2)
- added U5: MCP2562FDT-H_SN, Package_SO:SOIC-8_3.9x4.9mm_P1.27mm, B.Cu at (72.8, 192.5)
- added U6: MCP2562FDT-H_SN, Package_SO:SOIC-8_3.9x4.9mm_P1.27mm, B.Cu at (41.5, 194.0)
- added U7: TS30041, Package_DFN_QFN:QFN-16-1EP_3x3mm_P0.5mm_EP1.75x1.75mm_ThermalVias, B.Cu at (142.9, 76.4)
- added U8: MCP1700-3302E, Package_TO_SOT_SMD:SOT-23, B.Cu at (261.8, 82.5)
- added U9: ICM-20602, Package_LGA:LGA-16_3x3mm_P0.5mm_LayoutBorder3x5y, B.Cu at (220.4, 90.1)
- added X1: TXC-7C, Oscillator:Oscillator_SMD_TXC_7C-4Pin_5.0x3.2mm, B.Cu at (179.5, 82.0)
- C1, C2: value 1u -> 100n; footprint Capacitor_SMD:C_0805_2012Metric -> Capacitor_SMD:C_0603_1608Metric; moved to B.Cu
- C3: value 1u -> 2u2; footprint Capacitor_SMD:C_0805_2012Metric -> Capacitor_SMD:C_0603_1608Metric; moved to B.Cu
- C4: value 470m -> 100n; footprint Capacitor_SMD:CP_Elec_10x10.5 -> Capacitor_SMD:C_0603_1608Metric
- D1: value Schottky -> VIN; footprint Diode_SMD:D_SOD-123F -> LED_SMD:LED_0201_0603Metric
- J1: value UART -> Power In; footprint Connector_JST:JST_GH_BM04B-GHS-TBT_1x04-1MP_P1.25mm_Vertical -> TXV_Library_Footprints:Molex_MegaFit_1x03_Vertical
- J2: value GND -> Debug; footprint TestPoint:TestPoint_Pad_4.0x4.0mm -> Connector_PinHeader_2.54mm:PinHeader_1x08_P2.54mm_Vertical_SMD_Pin1Left
- J3: value ANT -> Debug; footprint TestPoint:TestPoint_THTPad_D1.5mm_Drill0.7mm -> Connector_PinHeader_1.27mm:PinHeader_2x04_P1.27mm_Vertical_SMD
- R1: value 330 -> 10k
- moved R1 103.6 mm to (231.2, 52.7), turned to 180 degrees
- moved C2 99.7 mm to (213.4, 34.5)
- moved C4 98.7 mm to (238.1, 66.3), turned to 180 degrees
- moved C3 93.8 mm to (221.2, 46.7), turned to 180 degrees
- moved D1 89.0 mm to (207.6, 42.2), turned to 180 degrees
- moved C1 76.4 mm to (158.6, 22.8), turned to 180 degrees
- moved J1 34.2 mm to (150.0, 65.8)
- moved J3 17.4 mm to (183.3, 115.5), turned to 180 degrees
- moved J2 0.52 mm to (185.8, 99.5), turned to 180 degrees
Connections:
- C2 pad 1: +3V3 -> GND
- C2 pad 2: GND -> +3V3
- C3 pad 1: Net-(C3-Pad1) -> GND
- C3 pad 2: GND -> +3V3
- C4 pad 1: Net-(C3-Pad1) -> GND
- C4 pad 2: GND -> +3V3
- D1 pad 1: Net-(D1-Pad1) -> GND
- D1 pad 2: +3V3 -> Net-(D1-Pad2)
- J1 pad 1: +3V3 -> +12V
- J1 pad 2: /TxD -> GND
- J1 pad 3: /RxD -> unconnected-(J1-Pad3)
- J2 pad 1: GND -> +3V3
- J3 pad 1: Net-(J3-Pad1) -> GND
- R1 pad 1: Net-(D1-Pad1) -> +3V3
- R1 pad 2: Net-(C3-Pad1) -> Net-(R1-Pad2)
- U1 pad 12: Net-(U1-Pad12) -> unconnected-(U1-Pad12)
- U1 pad 13: /TxD -> /GNSS_UART1_TX
- U1 pad 14: /RxD -> /GNSS_UART1_RX
- U1 pad 17: +3V3 -> Net-(C15-Pad2)
- U1 pad 19: Net-(U1-Pad19) -> /GNSS_INT
- U1 pad 2: +3V3 -> Net-(C15-Pad2)
- U1 pad 3: Net-(C3-Pad1) -> Net-(R9-Pad2)
- U1 pad 7: Net-(U1-Pad7) -> /GNSS_TPLS
- U1 pad 8: Net-(U1-Pad8) -> unconnected-(U1-Pad8)
- U1 pad 9: Net-(U1-Pad9) -> unconnected-(U1-Pad9)
Routing:
- net +3V3: track 31.7 -> 0.00 mm, vias 2 -> 0
- net Net-(C3-Pad1): track 12.3 -> 0.00 mm, vias 1 -> 0
- net /RxD: track 9.08 -> 0.00 mm, vias 1 -> 0
- net /TxD: track 8.81 -> 0.00 mm, vias 1 -> 0
- net Net-(D1-Pad1): track 1.58 -> 0.00 mm
- net GND: vias 54 -> 0
Other:
- net class Default removed
- board text removed: "GND RxD TxD 3V3"

Commit message: Updated layout; global placement done
Parts:
- removed F1: 500mA, Fuse:Fuse_0603_1608Metric
- added U10: LoRa1278F30, TXV_Library_Footprints:G-NiceRF-LoRa1278F30, B.Cu at (171.8, 103.3)
- D1, D3, D5: footprint LED_SMD:LED_0201_0603Metric -> LED_SMD:LED_0603_1608Metric
- J11, J5, J7, J9: value CAN1 -> CAN2
- moved C8 143.4 mm to (160.7, 69.5), turned to 180 degrees
- moved R11 133.8 mm to (132.0, 100.0), turned to 180 degrees
- moved D2 129.9 mm to (143.4, 113.3), turned to 90 degrees
- moved C14 129.6 mm to (135.5, 102.8), turned to -90 degrees
- moved U6 127.0 mm to (132.0, 104.8), turned to 90 degrees
- moved C17 124.3 mm to (135.5, 106.9), turned to 90 degrees
- moved R10 121.8 mm to (131.7, 88.8), turned to 180 degrees
- moved C13 116.6 mm to (135.5, 91.9), turned to -90 degrees
- moved U5 115.0 mm to (131.7, 93.7), turned to 90 degrees
- moved C16 111.0 mm to (135.5, 95.7), turned to -90 degrees
- moved C27 109.7 mm to (136.9, 77.7), turned to 0 degrees
- moved Q1 106.1 mm to (131.7, 79.7), turned to 90 degrees
- moved R9 105.4 mm to (145.4, 113.2), turned to 90 degrees
- moved JP1 101.3 mm to (102.4, 89.8)
- moved C7 100.0 mm to (148.7, 87.6)
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Connections:
- C16 pad 1: /5V_unfused -> +5V
- C17 pad 1: /5V_unfused -> +5V
- C23 pad 1: /5V_unfused -> +5V
- C24 pad 1: /5V_unfused -> +5V
- C25 pad 1: /5V_unfused -> +5V
- J10 pad 1: +5V -> Net-(J10-Pad1)
- J8 pad 1: +5V -> Net-(J10-Pad1)
- L1 pad 2: /5V_unfused -> +5V
- R12 pad 1: /5V_unfused -> +5V
- U5 pad 3: /5V_unfused -> +5V
- U6 pad 3: /5V_unfused -> +5V
- U8 pad 3: /5V_unfused -> +5V
Routing:
- net +5V: track 0.00 -> 61.0 mm
- net +3V3: track 0.00 -> 35.2 mm, vias 0 -> 1
- net Net-(C15-Pad2): track 0.00 -> 32.1 mm, vias 0 -> 2
- net /QSPI1_BK1_IO3: track 0.00 -> 16.7 mm
- net /CAN2_L: track 0.00 -> 15.1 mm
- net /CAN1_L: track 0.00 -> 14.9 mm
- net /QSPI1_CLK: track 0.00 -> 14.4 mm, vias 0 -> 2
- net Net-(R9-Pad2): track 0.00 -> 13.9 mm, vias 0 -> 1
- net /QSPI1_BK1_IO0: track 0.00 -> 13.1 mm
- net Net-(J12-PadS1): track 0.00 -> 13.0 mm
- net /GNSS_UART1_TX: track 0.00 -> 9.64 mm, vias 0 -> 1
- net /QSPI1_BK1_NCS: track 0.00 -> 9.46 mm, vias 0 -> 2
- net /GNSS_UART1_RX: track 0.00 -> 9.16 mm, vias 0 -> 1
- net /QSPI1_BK1_IO1: track 0.00 -> 8.82 mm, vias 0 -> 2
- net /CAN2_H: track 0.00 -> 8.13 mm
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Other:
- copper layers 2 -> 4
- board text added: "12V"
- board text added: "3V3"
- board text added: "5V"

Commit message: Update layout further
Parts:
- removed TP1, TP10, TP11, TP12, TP2, TP3, TP4, TP5, TP6, TP7, TP8, TP9: TestPoint_Probe, TestPoint:TestPoint_Pad_D1.0mm
- added G***: LOGO, TXV_Library_Footprints:ST_Logo_new, B.Cu at (145.9, 117.8)
- C31: value 100n -> 10n
- moved R3 106.2 mm to (138.6, 89.8), turned to -90 degrees
- moved J3 103.3 mm to (134.8, 100.0), turned to 180 degrees
- moved R2 96.3 mm to (143.4, 89.8), turned to -90 degrees
- moved LED1 90.6 mm to (145.2, 89.8), turned to 90 degrees
- moved R16 85.3 mm to (149.0, 69.8)
- moved R7 79.5 mm to (152.3, 68.0)
- moved R15 77.5 mm to (152.3, 69.8)
- moved LED2 73.6 mm to (140.3, 89.8), turned to 90 degrees
- moved R8 62.3 mm to (149.0, 68.0)
- moved D4 61.5 mm to (161.2, 83.0), turned to -90 degrees
- moved J2 39.9 mm to (119.5, 100.0), turned to -90 degrees
- moved JP1 38.1 mm to (140.1, 95.2), turned to -90 degrees
- moved D2 23.1 mm to (155.6, 93.7), turned to -90 degrees
- moved R9 22.9 mm to (157.4, 93.7), turned to -90 degrees
- moved R1 18.9 mm to (146.7, 68.8), turned to -90 degrees
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Connections:
- J10 pad 1: Net-(J10-Pad1) -> +5V
- J8 pad 1: Net-(J10-Pad1) -> +5V
Routing:
- net +5V: track 61.0 -> 197.7 mm, vias 0 -> 5
- net +3V3: track 35.2 -> 144.8 mm, vias 1 -> 9
- net /LoRa_SPI2_SCK: track 0.00 -> 55.1 mm, vias 0 -> 2
- net +12V: track 0.00 -> 54.5 mm
- net /LoRa_SPI2_MISO: track 0.00 -> 52.3 mm, vias 0 -> 2
- net /LoRa_SPI2_MOSI: track 0.00 -> 49.6 mm, vias 0 -> 2
- net /LoRa_SPI2_NSS: track 0.00 -> 48.3 mm, vias 0 -> 2
- net /LoRa_RST: track 0.00 -> 35.9 mm
- net /GNSS_INT: track 1.14 -> 26.5 mm, vias 0 -> 1
- net /SWCLK: track 0.00 -> 25.2 mm, vias 0 -> 2
- net /CAN1_H: track 7.96 -> 32.4 mm
- net /CAN2_H: track 8.13 -> 31.9 mm
- net /5V_PGOOD: track 0.00 -> 23.3 mm, vias 0 -> 2
- net /GNSS_TPLS: track 1.33 -> 22.2 mm, vias 0 -> 2
- net /GNSS_NRST: track 0.00 -> 18.8 mm, vias 0 -> 2
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- added copper zone on In1.Cu, net GND
Other:
- board text added: "1"
- board text added: "CAN1"
- board text added: "CAN2"
- board text added: "Debug"
- board text added: "Fabio Schartmüller"
- board text added: "INRCU v0.1"
- board text added: "Power State"
- board text added: "Status"

Commit message: Finished 1st proper layout
Parts:
- moved J12 40.1 mm to (158.6, 117.9), turned to 0 degrees
- moved C30 37.0 mm to (186.8, 112.7), turned to 0 degrees
- moved C29 36.6 mm to (186.8, 114.2), turned to 0 degrees
- moved G*** 6.19 mm to (142.0, 113.0)
- moved U10 0.77 mm to (173.1, 103.8), turned to 90 degrees
- moved C22 0.36 mm to (171.6, 68.2)
- moved D2 0.25 mm to (155.8, 93.7)
- moved R9 0.25 mm to (157.6, 93.7)
- moved Q1 0.10 mm to (132.4, 79.2)
- moved R4 0.10 mm to (132.3, 82.0)
Routing:
- net +3V3: track 144.8 -> 236.4 mm, vias 9 -> 13
- net +5V: track 197.7 -> 258.6 mm, vias 5 -> 10
- net /LoRa_DIO3: track 0.00 -> 52.9 mm, vias 0 -> 2
- net /LoRa_DIO5: track 0.00 -> 51.5 mm, vias 0 -> 2
- net /LoRa_DIO4: track 0.00 -> 49.8 mm, vias 0 -> 2
- net /LoRa_DIO0: track 0.00 -> 48.6 mm, vias 0 -> 2
- net /LoRa_DIO1: track 0.00 -> 47.5 mm, vias 0 -> 2
- net /CAN2_RX: track 0.00 -> 43.7 mm, vias 0 -> 2
- net /LoRa_DIO2: track 0.00 -> 42.1 mm, vias 0 -> 2
- net /LoRa_SPI2_SCK: track 55.1 -> 14.0 mm, vias 2 -> 0
- net /CAN2_TX: track 0.00 -> 39.8 mm, vias 0 -> 2
- net /UART_RX: track 4.50 -> 35.1 mm, vias 0 -> 2
- net /LoRa_SPI2_MISO: track 52.3 -> 22.3 mm
- net /LoRa_SPI2_MOSI: track 49.6 -> 22.0 mm, vias 2 -> 0
- net +12V: track 54.5 -> 82.0 mm, vias 0 -> 3
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Other:
- board text added: "GNSS"
- board text added: "LoRa asym HF"
- board text added: "System State"
- board text added: "maybe cut out for wiring X X X X X X X"
- board text added: "min GND Plane for internal patch antenna"
- board text removed: "Status"

Commit message: Update (in)official board name INRCU -> IMRCU
Other:
- board text added: "IMRCU v0.1"
- board text removed: "INRCU v0.1"
Changed lines of the file:
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@@
     (effects (font (size 1 1) (thickness 0.15)) (justify mirror))
   )
-  (gr_text "INRCU v0.1" (at 141 120.952) (layer "B.SilkS")
+  (gr_text "IMRCU v0.1" (at 141 120.952) (layer "B.SilkS")
     (effects (font (size 2 2) (thickness 0.5)) (justify mirror))
   )
@@
     (pts (xy 176.9 73.1) (xy 150 100))
     (height 13.788582)
-    (gr_text "38,0423 mm" (at 152.886827 75.986827 45) (layer "Dwgs.User")
+    (gr_text "38.0423 mm" (at 152.886827 75.986827 45) (layer "Dwgs.User")
       (effects (font (size 1 1) (thickness 0.15)))
     )
@@
   (segment (start 142.1185 83.168) (end 141.406 83.168) (width 0.2) (layer "B.Cu") (net 2))
   (segment (start 157.328 78.168) (end 157.62 77.876) (width 0.2) (layer "B.Cu") (net 2))
+  (segment (start 162.877989 81.345511) (end 162.5245 81.699) (width 0.5) (layer "B.Cu") (net 2))
   (segment (start 173.622 77.5595) (end 173.876 77.8135) (width 0.3) (layer "B.Cu") (net 2))
+  (segment (start 164.305489 81.345511) (end 162.877989 81.345511) (width 0.5) (layer "B.Cu") (net 2))
   (segment (start 140.094 73.584) (end 140.094 74.32) (width 0.3) (layer "B.Cu") (net 2))
   (segment (start 148.717 87.554) (end 148.73 87.554) (width 0.2) (layer "B.Cu") (net 2))
@@
   (segment (start 140.107 70.269) (end 140.107 71.057) (width 0.3) (layer "B.Cu") (net 2))
   (segment (start 157.62 77.051) (end 157.62 77.876) (width 0.3) (layer "B.Cu") (net 2))
-  (segment (start 164.305489 81.345511) (end 162.877989 81.345511) (width 0.5) (layer "B.Cu") (net 2))
   (segment (start 156.279 69.311) (end 156.279 68.066) (width 0.3) (layer "B.Cu") (net 2))
   (segment (start 155.4935 77.668) (end 156.475 77.668) (width 0.2) (layer "B.Cu") (net 2))
@@
   (segment (start 158.102 67.716) (end 158.128 67.742) (width 0.5) (layer "B.Cu") (net 2))
   (segment (start 137.643 76.632) (end 137.643 79.413) (width 0.2) (layer "B.Cu") (net 2))
-  (segment (start 164.381 81.27) (end 164.305489 81.345511) (width 0.5) (layer "B.Cu") (net 2))
   (segment (start 131.82724 89.434431) (end 131.966 89.295671) (width 0.3) (layer "B.Cu") (net 2))
   (segment (start 141.618 67.912) (end 141.618 70.112) (width 0.5) (layer "B.Cu") (net 2))
@@
   (segment (start 158.102 67.716) (end 159.639 67.716) (width 0.5) (layer "B.Cu") (net 2))
   (segment (start 162.059 81.699) (end 162.5245 81.699) (width 0.3) (layer "B.Cu") (net 2))
+  (segment (start 164.381 81.27) (end 164.305489 81.345511) (width 0.5) (layer "B.Cu") (net 2))
   (segment (start 137.643 79.413) (end 137.656 79.426) (width 0.2) (layer "B.Cu") (net 2))
   (segment (start 151.864258 73.21752) (end 151.556 72.909262) (width 0.2) (layer "B.Cu") (net 2))
@@
   (segment (start 173.622 76.886) (end 173.622 77.5595) (width 0.3) (layer "B.Cu") (net 2))
   (segment (start 131.204 97.968) (end 131.331 98.095) (width 0.3) (layer "B.Cu") (net 2))
-  (segment (start 162.877989 81.345511) (end 162.5245 81.699) (width 0.5) (layer "B.Cu") (net 2))
   (segment (start 131.101569 89.434431) (end 131.82724 89.434431) (width 0.3) (layer "B.Cu") (net 2))
   (segment (start 153.556 85.6055) (end 153.556 86.208) (width 0.2) (layer "B.Cu") (net 2))
